File: Project-1-ESP32-Environmental-Monitor/hardware/ESP32-Environmental-Monitor/ESP32-Environmental-Monitor.kicad_sch (KiCad schematic)
At the start: 5 parts, among them U1 AM2302, U2 ESP32-WROOM-32

Commit message: Add PCB layout and Gerber files
Parts:
- D1: footprint (none) -> LED_SMD:LED_0805_2012Metric
- R1, R2: footprint (none) -> Resistor_SMD:R_0805_2012Metric
Changed lines of the file:
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@@
 			)
 		)
-		(property "Footprint" ""
+		(property "Footprint" "Resistor_SMD:R_0805_2012Metric"
 			(at 169.672 90.17 90)
 			(hide yes)
@@
 			)
 		)
-		(property "Footprint" ""
+		(property "Footprint" "Resistor_SMD:R_0805_2012Metric"
 			(at 247.142 100.33 90)
 			(hide yes)
@@
 			)
 		)
-		(property "Footprint" ""
+		(property "Footprint" "LED_SMD:LED_0805_2012Metric"
 			(at 157.48 130.81 0)
 			(hide yes)
